File: electronics/hardware/jms_core_pcb/can.kicad_sch (KiCad schematic)
At the start: 9 parts

Commit message: Board Design - prototype now ordered
Parts:
- C1, C2, C3, C4: renamed from C?; footprint (none) -> Capacitor_THT:C_Disc_D5.0mm_W2.5mm_P5.00mm
- J5: renamed from J?; footprint (none) -> Connector_PinHeader_2.54mm:PinHeader_1x02_P2.54mm_Vertical
- R3: renamed from R?; footprint (none) -> Resistor_THT:R_Axial_DIN0207_L6.3mm_D2.5mm_P7.62mm_Horizontal
- U1: renamed from U?; value MCP2515-xSO -> MCP2515
- U2: renamed from U?; value MCP2561-E-P -> MCP2561
- Y1: renamed from Y?; footprint (none) -> Crystal:Crystal_HC49-U_Vertical
Connections:
- net CANH renamed CAN+
- net CANL renamed CAN-
Changed lines of the file:
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@@
     (effects (font (size 1.27 1.27)) (justify right bottom))
   )
-  (hierarchical_label "CANL" (shape output) (at 187.96 54.61 270)
-    (effects (font (size 1.27 1.27)) (justify right))
-  )
-  (hierarchical_label "CANH" (shape output) (at 187.96 44.45 90)
+  (hierarchical_label "CAN-" (shape output) (at 187.96 54.61 270)
+    (effects (font (size 1.27 1.27)) (justify right))
+  )
+  (hierarchical_label "CAN+" (shape output) (at 187.96 44.45 90)
     (effects (font (size 1.27 1.27)) (justify left))
   )
@@
   (symbol (lib_id "power:GND") (at 152.4 54.61 0) (unit 1)
     (in_bom yes) (on_board yes) (fields_autoplaced)
-    (property "Reference" "#PWR?" (id 0) (at 152.4 60.96 0)
+    (property "Reference" "#PWR022" (id 0) (at 152.4 60.96 0)
       (effects (font (size 1.27 1.27)) hide)
     )
@@
   (symbol (lib_id "power:+5V") (at 93.98 35.56 0) (unit 1)
     (in_bom yes) (on_board yes) (fields_autoplaced)
-    (property "Reference" "#PWR?" (id 0) (at 93.98 39.37 0)
+    (property "Reference" "#PWR020" (id 0) (at 93.98 39.37 0)
       (effects (font (size 1.27 1.27)) hide)
     )
@@
   (symbol (lib_id "power:GND") (at 55.88 73.66 0) (unit 1)
     (in_bom yes) (on_board yes) (fields_autoplaced)
-    (property "Reference" "#PWR?" (id 0) (at 55.88 80.01 0)
+    (property "Reference" "#PWR018" (id 0) (at 55.88 80.01 0)
       (effects (font (size 1.27 1.27)) hide)
     )
@@
   (symbol (lib_id "Connector_Generic:Conn_01x02") (at 203.2 48.26 0) (unit 1)
     (in_bom yes) (on_board yes) (fields_autoplaced)
-    (property "Reference" "J?" (id 0) (at 205.232 48.6215 0)
+    (property "Reference" "J5" (id 0) (at 205.232 48.6215 0)
       (effects (font (size 1.27 1.27)) (justify left))
     )
@@
       (effects (font (size 1.27 1.27)) (justify left))
     )
-    (property "Footprint" "" (id 2) (at 203.2 48.26 0)
+    (property "Footprint" "Connector_PinHeader_2.54mm:PinHeader_1x02_P2.54mm_Vertical" (id 2) (at 203.2 48.26 0)
       (effects (font (size 1.27 1.27)) hide)
     )
@@
   (symbol (lib_id "Device:R_Small") (at 194.31 46.99 90) (unit 1)
     (in_bom yes) (on_board yes) (fields_autoplaced)
-    (property "Reference" "R?" (id 0) (at 194.31 42.2869 90))
+    (property "Reference" "R3" (id 0) (at 194.31 42.2869 90))
     (property "Value" "120" (id 1) (at 194.31 45.062 90))
-    (property "Footprint" "" (id 2) (at 194.31 46.99 0)
+    (property "Footprint" "Resistor_THT:R_Axial_DIN0207_L6.3mm_D2.5mm_P7.62mm_Horizontal" (id 2) (at 194.31 46.99 0)
       (effects (font (size 1.27 1.27)) hide)
     )
@@
   (symbol (lib_id "power:GND") (at 165.1 59.69 0) (unit 1)
     (in_bom yes) (on_board yes) (fields_autoplaced)
-    (property "Reference" "#PWR?" (id 0) (at 165.1 66.04 0)
+    (property "Reference" "#PWR025" (id 0) (at 165.1 66.04 0)
       (effects (font (size 1.27 1.27)) hide)
     )
@@
   (symbol (lib_id "Device:Crystal") (at 67.31 66.04 270) (unit 1)
     (in_bom yes) (on_board yes) (fields_autoplaced)
-    (property "Reference" "Y?" (id 0) (at 70.6374 65.1315 90)
+    (property "Reference" "Y1" (id 0) (at 70.6374 65.1315 90)
       (effects (font (size 1.27 1.27)) (justify left))
     )
@@
       (effects (font (size 1.27 1.27)) (justify left))
     )
-    (property "Footprint" "" (id 2) (at 67.31 66.04 0)
+    (property "Footprint" "Crystal:Crystal_HC49-U_Vertical" (id 2) (at 67.31 66.04 0)
       (effects (font (size 1.27 1.27)) hide)
     )
@@
   (symbol (lib_id "power:GND") (at 83.82 36.83 0) (unit 1)
     (in_bom yes) (on_board yes)
-    (property "Reference" "#PWR?" (id 0) (at 83.82 43.18 0)
+    (property "Reference" "#PWR019" (id 0) (at 83.82 43.18 0)
       (effects (font (size 1.27 1.27)) hide)
     )
@@
   (symbol (lib_id "Device:C_Small") (at 86.36 36.83 90) (unit 1)
     (in_bom yes) (on_board yes) (fields_autoplaced)
-    (property "Reference" "C?" (id 0) (at 86.3663 31.3014 90))
+    (property "Reference" "C3" (id 0) (at 86.3663 31.3014 90))
     (property "Value" "0.1uF" (id 1) (at 86.3663 34.0765 90))
-    (property "Footprint" "" (id 2) (at 86.36 36.83 0)
+    (property "Footprint" "Capacitor_THT:C_Disc_D5.0mm_W2.5mm_P5.00mm" (id 2) (at 86.36 36.83 0)
       (effects (font (size 1.27 1.27)) hide)
     )
@@
   (symbol (lib_id "Interface_CAN_LIN:MCP2561-E-P") (at 165.1 49.53 0) (unit 1)
     (in_bom yes) (on_board yes) (fields_autoplaced)
-    (property "Reference" "U?" (id 0) (at 167.1194 37.9435 0)
-      (effects (font (size 1.27 1.27)) (justify left))
-    )
-    (property "Value" "MCP2561-E-P" (id 1) (at 167.1194 40.7186 0)
+    (property "Reference" "U2" (id 0) (at 167.1194 36.83 0)
+      (effects (font (size 1.27 1.27)) (justify left))
+    )
+    (property "Value" "MCP2561" (id 1) (at 167.1194 39.37 0)
       (effects (font (size 1.27 1.27)) (justify left))
     )
@@
   (symbol (lib_id "Interface_CAN_LIN:MCP2515-xSO") (at 93.98 59.69 0) (unit 1)
     (in_bom yes) (on_board yes) (fields_autoplaced)
-    (property "Reference" "U?" (id 0) (at 95.9994 37.9435 0)
-      (effects (font (size 1.27 1.27)) (justify left))
-    )
-    (property "Value" "MCP2515-xSO" (id 1) (at 95.9994 40.7186 0)
+    (property "Reference" "U1" (id 0) (at 95.9994 37.9435 0)
+      (effects (font (size 1.27 1.27)) (justify left))
+    )
+    (property "Value" "MCP2515" (id 1) (at 95.9994 40.7186 0)
       (effects (font (size 1.27 1.27)) (justify left))
     )
@@
   (symbol (lib_id "power:+5V") (at 165.1 35.56 0) (unit 1)
     (in_bom yes) (on_board yes) (fields_autoplaced)
-    (property "Reference" "#PWR?" (id 0) (at 165.1 39.37 0)
+    (property "Reference" "#PWR024" (id 0) (at 165.1 39.37 0)
       (effects (font (size 1.27 1.27)) hide)
     )
@@
   (symbol (lib_id "power:GND") (at 93.98 80.01 0) (unit 1)
     (in_bom yes) (on_board yes) (fields_autoplaced)
-    (property "Reference" "#PWR?" (id 0) (at 93.98 86.36 0)
+    (property "Reference" "#PWR021" (id 0) (at 93.98 86.36 0)
       (effects (font (size 1.27 1.27)) hide)
     )
@@
   (symbol (lib_id "Device:C") (at 59.69 62.23 90) (unit 1)
     (in_bom yes) (on_board yes) (fields_autoplaced)
-    (property "Reference" "C?" (id 0) (at 59.69 56.1045 90))
+    (property "Reference" "C1" (id 0) (at 59.69 56.1045 90))
     (property "Value" "22pF" (id 1) (at 59.69 58.8796 90))
-    (property "Footprint" "" (id 2) (at 63.5 61.2648 0)
+    (property "Footprint" "Capacitor_THT:C_Disc_D5.0mm_W2.5mm_P5.00mm" (id 2) (at 63.5 61.2648 0)
       (effects (font (size 1.27 1.27)) hide)
     )
@@
   (symbol (lib_id "Device:C_Small") (at 158.75 36.83 90) (unit 1)
     (in_bom yes) (on_board yes) (fields_autoplaced)
-    (property "Reference" "C?" (id 0) (at 158.7563 31.3014 90))
+    (property "Reference" "C4" (id 0) (at 158.7563 31.3014 90))
     (property "Value" "0.1uF" (id 1) (at 158.7563 34.0765 90))
-    (property "Footprint" "" (id 2) (at 158.75 36.83 0)
+    (property "Footprint" "Capacitor_THT:C_Disc_D5.0mm_W2.5mm_P5.00mm" (id 2) (at 158.75 36.83 0)
       (effects (font (size 1.27 1.27)) hide)
     )
@@
   (symbol (lib_id "Device:C") (at 59.69 69.85 90) (mirror x) (unit 1)
     (in_bom yes) (on_board yes)
-    (property "Reference" "C?" (id 0) (at 59.69 73.66 90))
+    (property "Reference" "C2" (id 0) (at 59.69 73.66 90))
     (property "Value" "22pF" (id 1) (at 59.69 66.4996 90))
-    (property "Footprint" "" (id 2) (at 63.5 70.8152 0)
+    (property "Footprint" "Capacitor_THT:C_Disc_D5.0mm_W2.5mm_P5.00mm" (id 2) (at 63.5 70.8152 0)
       (effects (font (size 1.27 1.27)) hide)
     )
@@
   (symbol (lib_id "power:GND") (at 156.21 36.83 0) (unit 1)
     (in_bom yes) (on_board yes)
-    (property "Reference" "#PWR?" (id 0) (at 156.21 43.18 0)
-      (effects (font (size 1.27 1.27)) hide)
-    )
+    (property "Reference" "#PWR023" (id 0) (at 156.21 43.18 0)
+      (effects (font (size 1.27 1.27)) hide)
+    )
