File: electronics/hardware/jms_core_pcb/jms_core_pcb.kicad_sch (KiCad schematic)
At the start: 4 parts

Commit message: Board Design - prototype now ordered
Parts:
- added D2: LED, LED_THT:LED_D3.0mm, symbol Device:LED
- added J13: Conn_01x03, TerminalBlock_Phoenix:TerminalBlock_Phoenix_MKDS-1,5-3-5.08_1x03_P5.08mm_Horizontal, symbol Connector_Generic:Conn_01x03
- added J14, J15: Conn_01x02, Connector_PinHeader_2.54mm:PinHeader_1x02_P2.54mm_Vertical, symbol Connector_Generic:Conn_01x02
- added J2: IO_BREAK, Connector_PinHeader_2.54mm:PinHeader_2x10_P2.54mm_Vertical, symbol Connector_Generic:Conn_02x10_Odd_Even
- added J3, J4: RJ45, Connector_RJ:RJ45_Amphenol_54602-x08_Horizontal, symbol Connector:RJ45
- added R4: 120, Resistor_THT:R_Axial_DIN0207_L6.3mm_D2.5mm_P7.62mm_Horizontal, symbol Device:R_Small
- D1: footprint (none) -> LED_THT:LED_D3.0mm
- J1: renamed from J?; footprint (none) -> Connector_PinHeader_2.54mm:PinHeader_1x02_P2.54mm_Vertical
- R1, R2: renamed from R?; footprint (none) -> Resistor_THT:R_Axial_DIN0207_L6.3mm_D2.5mm_P7.62mm_Horizontal
Connections:
- net +5V: now also D2.2 (A), J13.1 (Pin_1), J14.2 (Pin_2), J15.2 (Pin_2), J2.1 (Pin_1)
- net AI0: now also J2.15 (Pin_15)
- net AI1: now also J2.16 (Pin_16)
- net AI2: now also J2.18 (Pin_18)
- net DIO4: now also J2.4 (Pin_4)
- net DIO5: now also J2.6 (Pin_6)
- net DIO6: now also J2.8 (Pin_8)
- net DIO7: now also J2.10 (Pin_10)
- net DIO8: now also J2.12 (Pin_12)
- net DIO9: now also J2.14 (Pin_14)
- net GND: now also J13.3 (Pin_3), J2.17 (Pin_17), J2.19 (Pin_19), J2.20 (Pin_20), J3.1, J4.1, R4.2
- net I2C_SCL: now also J2.5 (Pin_5)
- net I2C_SDA: now also J2.3 (Pin_3)
- net MASTER_SEL: now also J2.13 (Pin_13)
- net RESET: now also J2.11 (Pin_11)
- new net: J14.1 (Pin_1), J4.2
- new net: J15.1 (Pin_1), J3.2
- new net: D2.1 (K), R4.1
- new net +3V3: J13.2 (Pin_2), J2.2 (Pin_2)
- new net CAN+: J2.7 (Pin_7), J3.8, J4.8
- new net CAN-: J2.9 (Pin_9), J3.7, J4.7
Other:
- added sheet driver_station (driver_station.kicad_sch)
- sheet CAN ports: added CAN+, CAN-; removed CANH, CANL
- sheet Master ports: added CAN+, CAN-; removed CANH, CANL
- note added: "MASTER/DS: FIELD 1 FIELD: IN"
- note added: "MASTER/DS: FIELD 2 FIELD: OUT"
