File: electronics/hardware/jms_core_pcb/master.kicad_sch (KiCad schematic)
At the start: 6 parts

Commit message: Board Design - prototype now ordered
Parts:
- removed J?: BLUE_ESTOP, symbol Connector_Generic:Conn_01x04
- removed J?: RED_ESTOP, symbol Connector_Generic:Conn_01x04
- removed J?: RJ45, symbol Connector:RJ45
- added D10, D11, D3, D4, D5, D6, D7, D8, D9: LED, LED_THT:LED_D3.0mm, symbol Device:LED
- added R10, R11, R12, R13, R5, R6, R7, R8, R9: 120, Resistor_THT:R_Axial_DIN0207_L6.3mm_D2.5mm_P7.62mm_Horizontal, symbol Device:R_Small
- J10, J9: renamed from J?; footprint (none) -> Connector_RJ:RJ45_Amphenol_54602-x08_Horizontal
- J6: renamed from J?; footprint (none) -> TerminalBlock_Phoenix:TerminalBlock_Phoenix_MKDS-1,5-2-5.08_1x02_P5.08mm_Horizontal
Connections:
- net +5V: now also D10.2 (A), D11.2 (A), D3.2 (A), D4.2 (A), D5.2 (A), D6.2 (A), D7.2 (A), D8.2 (A), D9.2 (A)
- net DETECT_BLUE: now also R9.2
- net DETECT_RED: now also R5.2
- net ESTOP_BLUE_1: now also R10.2
- net ESTOP_BLUE_2: now also R11.2
- net ESTOP_BLUE_3: now also R12.2
- net ESTOP_FIELD: now also R13.2
- net ESTOP_RED_1: now also R6.2
- net ESTOP_RED_2: now also R7.2
- net ESTOP_RED_3: now also R8.2
- net CANH renamed CAN+
- net CANL renamed CAN-
- new net: D9.1 (K), R11.1
- new net: D10.1 (K), R12.1
- new net: D8.1 (K), R10.1
- new net: D4.1 (K), R6.1
- new net: D5.1 (K), R7.1
- new net: D6.1 (K), R8.1
- new net: D3.1 (K), R5.1
- new net: D7.1 (K), R9.1
- new net: D11.1 (K), R13.1
Other:
- note added: "MASTER TO BLUE"
- note removed: "MASTER TO FIELD"
- moved on the sheet: J6
