File: electronics/hardware/jms_core_pcb/mcu_arduino.kicad_sch (KiCad schematic)
At the start: 2 parts

Commit message: Board Design - prototype now ordered
Parts:
- gave numbers to parts that had none: 2
Changed lines of the file:
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@@
   (symbol (lib_id "power:+3V3") (at 72.39 30.48 0) (unit 1)
     (in_bom yes) (on_board yes)
-    (property "Reference" "#PWR?" (id 0) (at 72.39 34.29 0)
+    (property "Reference" "#PWR014" (id 0) (at 72.39 34.29 0)
       (effects (font (size 1.27 1.27)) hide)
     )
@@
   (symbol (lib_id "power:+5V") (at 74.93 97.79 0) (unit 1)
     (in_bom yes) (on_board yes)
-    (property "Reference" "#PWR?" (id 0) (at 74.93 101.6 0)
+    (property "Reference" "#PWR017" (id 0) (at 74.93 101.6 0)
       (effects (font (size 1.27 1.27)) hide)
     )
@@
   (symbol (lib_id "MCU_Module:Arduino_Nano_v3.x") (at 69.85 123.19 0) (unit 1)
     (in_bom yes) (on_board yes) (fields_autoplaced)
-    (property "Reference" "A?" (id 0) (at 74.4094 148.1995 0)
+    (property "Reference" "A2" (id 0) (at 74.4094 148.1995 0)
       (effects (font (size 1.27 1.27)) (justify left))
     )
@@
   (symbol (lib_id "power:GND") (at 69.85 86.36 0) (unit 1)
     (in_bom yes) (on_board yes) (fields_autoplaced)
-    (property "Reference" "#PWR?" (id 0) (at 69.85 92.71 0)
+    (property "Reference" "#PWR012" (id 0) (at 69.85 92.71 0)
       (effects (font (size 1.27 1.27)) hide)
     )
@@
   (symbol (lib_id "power:GND") (at 71.12 151.13 0) (unit 1)
     (in_bom yes) (on_board yes) (fields_autoplaced)
-    (property "Reference" "#PWR?" (id 0) (at 71.12 157.48 0)
+    (property "Reference" "#PWR013" (id 0) (at 71.12 157.48 0)
       (effects (font (size 1.27 1.27)) hide)
     )
@@
   (symbol (lib_id "power:+3V3") (at 72.39 97.79 0) (unit 1)
     (in_bom yes) (on_board yes)
-    (property "Reference" "#PWR?" (id 0) (at 72.39 101.6 0)
+    (property "Reference" "#PWR015" (id 0) (at 72.39 101.6 0)
       (effects (font (size 1.27 1.27)) hide)
     )
@@
   (symbol (lib_id "power:+5V") (at 74.93 30.48 0) (unit 1)
     (in_bom yes) (on_board yes)
-    (property "Reference" "#PWR?" (id 0) (at 74.93 34.29 0)
+    (property "Reference" "#PWR016" (id 0) (at 74.93 34.29 0)
       (effects (font (size 1.27 1.27)) hide)
     )
@@
   (symbol (lib_id "MCU_Module:Arduino_UNO_R2") (at 69.85 55.88 0) (unit 1)
     (in_bom yes) (on_board yes) (fields_autoplaced)
-    (property "Reference" "A?" (id 0) (at 76.9494 29.0535 0)
+    (property "Reference" "A1" (id 0) (at 76.9494 29.0535 0)
       (effects (font (size 1.27 1.27)) (justify left))
     )
