File: electronics/hardware/jms_ufe_controller/dmx.kicad_sch (KiCad schematic)
At the start: 8 parts, among them J13 XLR3, U5 MAX485E

Commit message: UFE Rev 3 - first try
Parts:
- removed J13: XLR3, XLR:CONN-TH_DIN-313HF, symbol Connector:XLR3
- removed TP1, TP2, TP3: TestPoint, TestPoint:TestPoint_Pad_D2.0mm, symbol Connector:TestPoint
- added J1: Conn_01x03, symbol Connector_Generic:Conn_01x03
Connections:
- net DMX+: now also J1.3 (Pin_3)
- net DMX-: now also J1.2 (Pin_2)
- net GND: now also J1.1 (Pin_1)
Other:
- moved on the sheet: C27, C28, R15, U5
