File: electronics/hardware/jms_ufe_controller/jms_ufe_controller.kicad_pcb (KiCad board)
At the start: 4 copper layers, 100 x 70 mm, 94 parts, among them J1 Conn_02x03_Odd_Even, J11 RJ45_Amphenol_RJMG1BD3B8K1ANR, J12 TC2050-IDC-NL, J13 XLR3, J2 Conn_02x03_Odd_Even, J3 Conn_01x04, J4 Conn_01x04, J5 Conn_01x03, J6 Conn_01x04, J7 Conn_01x02, J8 Conn_01x02, J9 Conn_01x04, SW1 SW_DIP_x04, U1 STM32F407VGTx, U2 MCP1703Ax-500xxTT, U3 DP83848KSQ_NOPB, U4 MCP1703Ax-330xxTT, U5 MAX485E

Commit message: UFE Rev 2 off to the board fab
Parts:
- added D12: LED GREEN, LED_SMD:LED_0603_1608Metric, F.Cu at (168.2, 64.6)
- added D13: LED GREEN, LED_SMD:LED_0603_1608Metric, F.Cu at (164.6, 64.6)
- added D14: LED GREEN, LED_SMD:LED_0603_1608Metric, F.Cu at (161.1, 64.6)
- added D15: LED GREEN, LED_SMD:LED_0603_1608Metric, F.Cu at (157.5, 64.6)
- added D16: LED GREEN, LED_SMD:LED_0603_1608Metric, F.Cu at (154.0, 64.6)
- added D17: LED GREEN, LED_SMD:LED_0603_1608Metric, F.Cu at (150.4, 64.6)
- added D18: LED GREEN, LED_SMD:LED_0603_1608Metric, F.Cu at (146.9, 64.6)
- added D19: LED GREEN, LED_SMD:LED_0603_1608Metric, F.Cu at (143.3, 64.6)
- added G***: LOGO, LOGO, F.Cu at (154.5, 60.6)
- added G***: LOGO, LOGO, F.Cu at (180.9, 60.6)
- added G***: LOGO, LOGO, F.Cu at (131.6, 60.6)
- added G***: LOGO, LOGO, F.Cu at (187.0, 77.8)
- added G***: LOGO, LOGO, F.Cu at (176.3, 109.3)
- added G***: LOGO, LOGO, F.Cu at (162.9, 70.2)
- added G***: LOGO, LOGO, F.Cu at (116.6, 60.6)
- added G***: LOGO, LOGO, F.Cu at (156.8, 109.1)
- added G***: LOGO, LOGO, F.Cu at (149.7, 109.1)
- added Q1: LMUN2233LT1G, LMUN2233:SOT-23-3_L2.9-W1.6-P1.90-LS2.8-BR, F.Cu at (174.3, 101.2)
- added Q2: LMUN2233LT1G, LMUN2233:SOT-23-3_L2.9-W1.6-P1.90-LS2.8-BR, F.Cu at (170.7, 101.2)
- added Q3: LMUN2233LT1G, LMUN2233:SOT-23-3_L2.9-W1.6-P1.90-LS2.8-BR, F.Cu at (167.2, 101.2)
- added Q4: LMUN2233LT1G, LMUN2233:SOT-23-3_L2.9-W1.6-P1.90-LS2.8-BR, F.Cu at (163.6, 101.2)
- added Q5: LMUN2233LT1G, LMUN2233:SOT-23-3_L2.9-W1.6-P1.90-LS2.8-BR, F.Cu at (188.5, 101.2)
- added Q6: LMUN2233LT1G, LMUN2233:SOT-23-3_L2.9-W1.6-P1.90-LS2.8-BR, F.Cu at (185.0, 101.2)
- added Q7: LMUN2233LT1G, LMUN2233:SOT-23-3_L2.9-W1.6-P1.90-LS2.8-BR, F.Cu at (181.4, 101.2)
- added Q8: LMUN2233LT1G, LMUN2233:SOT-23-3_L2.9-W1.6-P1.90-LS2.8-BR, F.Cu at (177.9, 101.2)
- added R26: 220, Resistor_SMD:R_0402_1005Metric, F.Cu at (166.7, 65.1)
- added R27: 220, Resistor_SMD:R_0402_1005Metric, F.Cu at (163.1, 65.1)
- added R28: 220, Resistor_SMD:R_0402_1005Metric, F.Cu at (159.6, 65.1)
- added R29: 220, Resistor_SMD:R_0402_1005Metric, F.Cu at (156.0, 65.1)
- added R30: 220, Resistor_SMD:R_0402_1005Metric, F.Cu at (152.5, 65.1)
- added R31: 220, Resistor_SMD:R_0402_1005Metric, F.Cu at (148.9, 65.1)
- added R32: 220, Resistor_SMD:R_0402_1005Metric, F.Cu at (145.3, 65.1)
- added R33: 220, Resistor_SMD:R_0402_1005Metric, F.Cu at (141.8, 65.1)
- J3, J6: value Conn_01x04 -> Conn_01x08; footprint TerminalBlock_Phoenix:TerminalBlock_Phoenix_PT-1,5-4-5.0-H_1x04_P5.00mm_Horizontal -> TerminalBlock_Phoenix:TerminalBlock_Phoenix_PT-1,5-8-3.5-H_1x08_P3.50mm_Horizontal
- J4, J9: footprint TerminalBlock_Phoenix:TerminalBlock_Phoenix_PT-1,5-4-5.0-H_1x04_P5.00mm_Horizontal -> TerminalBlock_Phoenix:TerminalBlock_Phoenix_PT-1,5-4-3.5-H_1x04_P3.50mm_Horizontal
- J5: footprint TerminalBlock_Phoenix:TerminalBlock_Phoenix_PT-1,5-3-5.0-H_1x03_P5.00mm_Horizontal -> TerminalBlock_Phoenix:TerminalBlock_Phoenix_PT-1,5-3-3.5-H_1x03_P3.50mm_Horizontal
- J7, J8: footprint TerminalBlock_Phoenix:TerminalBlock_Phoenix_PT-1,5-2-5.0-H_1x02_P5.00mm_Horizontal -> TerminalBlock_Phoenix:TerminalBlock_Phoenix_PT-1,5-2-3.5-H_1x02_P3.50mm_Horizontal
- moved D11 50.9 mm to (177.3, 105.0), turned to -90 degrees
- moved R25 50.1 mm to (178.9, 104.5)
- moved D10 50.0 mm to (180.6, 105.0), turned to -90 degrees
- moved D9 49.2 mm to (184.2, 105.0), turned to -90 degrees
- moved R24 49.2 mm to (182.2, 104.5)
- moved D8 48.6 mm to (187.8, 105.0), turned to -90 degrees
- moved R23 48.5 mm to (185.7, 104.5)
- moved R22 47.9 mm to (189.3, 104.5)
- moved R21 26.7 mm to (164.4, 104.5), turned to -90 degrees
- moved D7 25.9 mm to (162.9, 105.0), turned to -90 degrees
- moved R20 18.5 mm to (167.9, 104.5), turned to -90 degrees
- moved D6 17.5 mm to (166.4, 105.0), turned to -90 degrees
- moved R19 10.4 mm to (171.5, 104.5), turned to -90 degrees
- moved J7 10.2 mm to (133.4, 55.2)
- moved J3 9.29 mm to (164.1, 114.7)
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Connections:
- net /DIN_1 renamed /Digital IO/DIN_1
- D10 pad 1: GND -> Net-(D10-Pad1)
- D11 pad 1: GND -> Net-(D11-Pad1)
- D4 pad 1: /DIN1_LED -> Net-(D4-Pad1)
- D5 pad 1: /DIN2_LED -> Net-(D5-Pad1)
- D6 pad 1: /DIN3_LED -> Net-(D6-Pad1)
- D7 pad 1: /DIN4_LED -> Net-(D7-Pad1)
- D8 pad 1: GND -> Net-(D8-Pad1)
- D9 pad 1: GND -> Net-(D9-Pad1)
- J3 pad 2: /DIN_2 -> /Digital IO/DIN_2
- J3 pad 3: /DIN_3 -> /Digital IO/DIN_3
- J3 pad 4: /DIN_4 -> /Digital IO/DIN_4
- J6 pad 1: /DOUT_1 -> /Digital IO/DOUT_1
- J6 pad 2: /DOUT_2 -> /Digital IO/DOUT_2
- J6 pad 3: /DOUT_3 -> /Digital IO/DOUT_3
- J6 pad 4: /DOUT_4 -> /Digital IO/DOUT_4
- R22 pad 1: /DOUT_1 -> +3V3
- R23 pad 1: /DOUT_2 -> +3V3
- R24 pad 1: /DOUT_3 -> +3V3
- R25 pad 1: /DOUT_4 -> +3V3
- U1 pad 39: /DIN1_LED -> /Digital IO/DIN_2
- U1 pad 40: /DIN_2 -> /Digital IO/DIN_3
- U1 pad 41: /DIN2_LED -> /Digital IO/DIN_4
- U1 pad 42: /DIN_3 -> /Digital IO/DIN_5
- U1 pad 43: /DIN3_LED -> /Digital IO/DIN_6
- U1 pad 44: /DIN_4 -> /Digital IO/DIN_7
- U1 pad 45: /DIN4_LED -> /Digital IO/DIN_8
- U1 pad 81: /DOUT_1 -> /Digital IO/DOUT_1
- U1 pad 82: /DOUT_2 -> /Digital IO/DOUT_2
- U1 pad 83: /DOUT_3 -> /Digital IO/DOUT_3
- U1 pad 84: /DOUT_4 -> /Digital IO/DOUT_4
- U1 pad 85: unconnected-(U1-Pad85) -> /Digital IO/DOUT_5
- U1 pad 86: unconnected-(U1-Pad86) -> /Digital IO/DOUT_6
- U1 pad 87: unconnected-(U1-Pad87) -> /Digital IO/DOUT_7
- U1 pad 88: unconnected-(U1-Pad88) -> /Digital IO/DOUT_8
Routing:
- net +3V3: track 374.4 -> 317.2 mm, vias 11 -> 19
- net /Digital IO/DIN_8: track 0.00 -> 45.7 mm
- net /Digital IO/DIN_7: track 0.00 -> 43.0 mm
- net /Digital IO/DIN_6: track 0.00 -> 40.0 mm
- net /DIN_4: track 39.9 -> 0.00 mm
- net /Digital IO/DOUT_8: track 0.00 -> 38.9 mm
- net /Digital IO/DIN_5: track 0.00 -> 37.0 mm
- net /DIN_3: track 36.0 -> 0.00 mm
- net /Digital IO/DOUT_7: track 0.00 -> 35.9 mm
- net /Digital IO/DIN_4: track 0.00 -> 34.0 mm
- net /DIN4_LED: track 33.6 -> 0.00 mm
- net /Digital IO/DOUT_6: track 0.00 -> 33.1 mm
- net /DIN_2: track 32.1 -> 0.00 mm
- net /Digital IO/DIN_3: track 0.00 -> 31.2 mm
- net /Digital IO/DOUT_5: track 0.00 -> 29.9 mm
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Other:
- board text removed: "+3V3"
- board text removed: "AI1"
- board text removed: "AI2"
- board text removed: "AI3"
- board text removed: "AI4"
- board text removed: "ANALOG IN"
- board text removed: "ANALOG OUT"
- board text removed: "AO1"
- board text removed: "AO2"
- board text removed: "DI1"
- board text removed: "DI2"
- board text removed: "DI3"
- board text removed: "DI4"
- board text removed: "DIGITAL IN"
- board text removed: "DIGITAL OUT"
- board text removed: "DO1"
- board text removed: "DO2"
- board text removed: "DO3"
- board text removed: "DO4"
- board text removed: "IN1"
- board text removed: "IN2"
- board text removed: "IN3"
- board text removed: "POWER OUT"
- board text removed: "PWM IN"
- board text removed: "PWM OUT"

Commit message: UFE Rev 3 - first try
Parts:
- removed D5, D6: LED GREEN, LED_SMD:LED_0603_1608Metric
- removed G*** (x9): LOGO, LOGO
- removed J11: RJ45_Amphenol_RJMG1BD3B8K1ANR, Connector_RJ:RJ45_Amphenol_RJMG1BD3B8K1ANR
- removed J12: TC2050-IDC-NL, Project:TAG-CONNECT_TC2050-IDC-NL
- removed J13: XLR3, XLR:CONN-TH_DIN-313HF
- removed J9: Conn_01x04, TerminalBlock_Phoenix:TerminalBlock_Phoenix_PT-1,5-4-3.5-H_1x04_P3.50mm_Horizontal
- removed Q1, Q2, Q3, Q4, Q5, Q6, Q7, Q8: LMUN2233LT1G, LMUN2233:SOT-23-3_L2.9-W1.6-P1.90-LS2.8-BR
- added C29: 0u1, Capacitor_SMD:C_0402_1005Metric, F.Cu at (89.0, -54.4)
- added C30: 0u1, Capacitor_SMD:C_0402_1005Metric, F.Cu at (76.3, -42.3)
- added C31: 4pF, Capacitor_SMD:C_0402_1005Metric, F.Cu at (79.2, -45.5)
- added C32: 0u1, Capacitor_SMD:C_0402_1005Metric, F.Cu at (79.2, -43.5)
- added C33: 4pF, Capacitor_SMD:C_0402_1005Metric, F.Cu at (94.5, -61.9)
- added C34: 0u1, Capacitor_SMD:C_0402_1005Metric, F.Cu at (73.1, -38.4)
- added C35: 0u1, Capacitor_SMD:C_0402_1005Metric, F.Cu at (73.1, -40.3)
- added C36: 0u1, Capacitor_SMD:C_0402_1005Metric, F.Cu at (97.4, -63.9)
- added C37: 0u1, Capacitor_SMD:C_0402_1005Metric, F.Cu at (103.9, -67.9)
- added C38: 0u1, Capacitor_SMD:C_0402_1005Metric, F.Cu at (101.0, -67.9)
- added C39: 0u1, Capacitor_SMD:C_0402_1005Metric, F.Cu at (86.1, -54.1)
- added C40: 0u1, Capacitor_SMD:C_0402_1005Metric, F.Cu at (88.5, -52.2)
- added C41: 0u1, Capacitor_SMD:C_0402_1005Metric, F.Cu at (82.8, -48.2)
- added C42: 0u1, Capacitor_SMD:C_0402_1005Metric, F.Cu at (100.3, -64.0)
- added C43: 0u1, Capacitor_SMD:C_0402_1005Metric, F.Cu at (97.4, -61.9)
- added C44: 0u1, Capacitor_SMD:C_0402_1005Metric, F.Cu at (96.6, -59.9)
- added C45: 0u1, Capacitor_SMD:C_0402_1005Metric, F.Cu at (103.9, -69.9)
- added C46: 0u1, Capacitor_SMD:C_0402_1005Metric, F.Cu at (76.3, -40.4)
- added C47: 0u1, Capacitor_SMD:C_0402_1005Metric, F.Cu at (70.2, -36.7)
- added C48: 0u1, Capacitor_SMD:C_0402_1005Metric, F.Cu at (85.7, -50.2)
- added C49: 10uF, Capacitor_SMD:C_0402_1005Metric, F.Cu at (73.1, -36.4)
- added C50: 0u1, Capacitor_SMD:C_0402_1005Metric, F.Cu at (82.8, -50.2)
- added C51: 0u1, Capacitor_SMD:C_0402_1005Metric, F.Cu at (85.6, -52.2)
- added C52: 0u1, Capacitor_SMD:C_0402_1005Metric, F.Cu at (101.0, -69.9)
- added C53: 0u1, Capacitor_SMD:C_0402_1005Metric, F.Cu at (93.7, -59.9)
- added C54: 0u1, Capacitor_SMD:C_0402_1005Metric, F.Cu at (91.9, -56.4)
- added C55: 0u1, Capacitor_SMD:C_0402_1005Metric, F.Cu at (85.7, -48.2)
- added C56: 0u1, Capacitor_SMD:C_0402_1005Metric, F.Cu at (82.8, -46.2)
- added C57: 22uF, Capacitor_SMD:C_0402_1005Metric, F.Cu at (90.8, -58.3)
- added C58: 0u1, Capacitor_SMD:C_0402_1005Metric, F.Cu at (70.2, -38.7)
- added C59: 0u1, Capacitor_SMD:C_0402_1005Metric, F.Cu at (101.0, -66.0)
- added C60: 0u1, Capacitor_SMD:C_0402_1005Metric, F.Cu at (66.9, -34.6)
- added C61: 0u1, Capacitor_SMD:C_0402_1005Metric, F.Cu at (89.0, -56.4)
- added C62: 10uF, Capacitor_SMD:C_0402_1005Metric, F.Cu at (103.7, -71.9)
- added C63: 0u1 100V, Capacitor_SMD:C_0805_2012Metric, F.Cu at (60.1, -38.7)
- added C64: 33uF, Capacitor_THT:CP_Radial_D16.0mm_P7.50mm, F.Cu at (116.1, -67.6)
- added C66: 22pF, Capacitor_SMD:C_0402_1005Metric, F.Cu at (155.0, -69.0)
- added C67: 22uF, Capacitor_SMD:C_0402_1005Metric, F.Cu at (126.5, -40.0)
- added C68: 22uF, Capacitor_SMD:C_0402_1005Metric, F.Cu at (132.9, -45.6)
- added C69: 22uF, Capacitor_SMD:C_0402_1005Metric, F.Cu at (145.4, -58.7)
- added C71: 1000uF low-ESR, Capacitor_THT:CP_Radial_D12.5mm_P5.00mm, F.Cu at (115.5, -39.5)
- added C72: 22pF, Capacitor_SMD:C_0402_1005Metric, F.Cu at (145.4, -60.7)
- added C73: 22uF, Capacitor_SMD:C_0402_1005Metric, F.Cu at (130.0, -43.7)
- added C74: 22uF, Capacitor_SMD:C_0402_1005Metric, F.Cu at (139.9, -53.2)
- added C75: 22uF, Capacitor_SMD:C_0402_1005Metric, F.Cu at (145.4, -62.7)
- added C76: 1uF, Capacitor_SMD:C_0402_1005Metric, F.Cu at (130.0, -45.6)
- added C77: 1uF, Capacitor_SMD:C_0402_1005Metric, F.Cu at (148.3, -62.7)
- added C78: 0u1, Capacitor_SMD:C_0402_1005Metric, F.Cu at (190.0, -98.6)
- added C79: 0u1, Capacitor_SMD:C_0402_1005Metric, F.Cu at (173.0, -82.8)
- added C80: 0u1, Capacitor_SMD:C_0402_1005Metric, F.Cu at (205.9, -118.5)
- added C81: 0u1, Capacitor_SMD:C_0402_1005Metric, F.Cu at (175.8, -82.8)
- added C82: 0u1, Capacitor_SMD:C_0402_1005Metric, F.Cu at (208.7, -116.5)
- added C83: 0u1, Capacitor_SMD:C_0402_1005Metric, F.Cu at (206.5, -114.6)
- added C84: 0u1, Capacitor_SMD:C_0402_1005Metric, F.Cu at (173.0, -80.8)
- added C85: 0u1, Capacitor_SMD:C_0402_1005Metric, F.Cu at (167.2, -80.8)
- added C86: 0u1, Capacitor_SMD:C_0402_1005Metric, F.Cu at (170.1, -82.8)
- added C87: 0u1, Capacitor_SMD:C_0402_1005Metric, F.Cu at (170.1, -80.8)
- added C88: 0u1, Capacitor_SMD:C_0402_1005Metric, F.Cu at (193.0, -100.6)
- added C89: 0u1, Capacitor_SMD:C_0402_1005Metric, F.Cu at (167.2, -82.8)
- added C90: 0u1, Capacitor_SMD:C_0402_1005Metric, F.Cu at (187.2, -98.6)
- added C91: 0u1, Capacitor_SMD:C_0402_1005Metric, F.Cu at (164.3, -80.8)
- added C92: 0u1, Capacitor_SMD:C_0402_1005Metric, F.Cu at (211.6, -118.5)
- added C93: 0u1, Capacitor_SMD:C_0402_1005Metric, F.Cu at (208.7, -118.5)
- added C94: 0u1, Capacitor_SMD:C_0402_1005Metric, F.Cu at (222.3, -129.6)
- added C95: 0u1, Capacitor_SMD:C_0402_1005Metric, F.Cu at (205.9, -116.5)
- added C96: 0u1, Capacitor_SMD:C_0402_1005Metric, F.Cu at (225.2, -131.6)
- added C97: 0u1, Capacitor_SMD:C_0402_1005Metric, F.Cu at (222.3, -131.6)
- added C98: 1uF, Capacitor_SMD:C_0402_1005Metric, F.Cu at (91.9, -83.7)
- added D20: SS210, Diode_SMD:D_SMA, F.Cu at (74.2, -56.3)
- added D21: DB207S_C29174, DB207S:DBS_L8.4-W6.4-P5.10-LS10.2-TL, F.Cu at (64.0, -53.7)
- added D22: LED_GREEN, LED_SMD:LED_0603_1608Metric, F.Cu at (80.2, -59.4)
- added D23: SMF58A, Diode_SMD:D_SMF, F.Cu at (78.6, -64.9)
- added D24: DB207S_C29174, DB207S:DBS_L8.4-W6.4-P5.10-LS10.2-TL, F.Cu at (81.8, -71.5)
- added D25: SS210, Diode_SMD:D_SMA, F.Cu at (147.4, -74.1)
- added L1: 2.2uH, Inductor_SMD:L_1008_2520Metric, F.Cu at (145.9, -65.5)
- added L2: 150uH, Inductor_SMD:L_12x12mm_H8mm, F.Cu at (136.0, -69.3)
- added L3: 2.2uH, Inductor_SMD:L_1008_2520Metric, F.Cu at (151.0, -70.0)
- added L4: G2406S_C507595, G2406S:SMD-24_L15.1-W7.1-P1.00-LS10.0-BL, F.Cu at (112.8, 107.0)
- added L5: G2406S_C507595, G2406S:SMD-24_L15.1-W7.1-P1.00-LS10.0-BL, F.Cu at (163.6, 106.3)
- added L6: G2406S_C507595, G2406S:SMD-24_L15.1-W7.1-P1.00-LS10.0-BL, F.Cu at (112.8, 87.2)
- added L7: G2406S_C507595, G2406S:SMD-24_L15.1-W7.1-P1.00-LS10.0-BL, F.Cu at (163.6, 87.2)
- added L8: G2406S_C507595, G2406S:SMD-24_L15.1-W7.1-P1.00-LS10.0-BL, F.Cu at (112.8, 66.9)
- added R34: 1k27 1%, Resistor_SMD:R_0402_1005Metric, F.Cu at (77.0, -49.5)
- added R35: 10k, Resistor_SMD:R_0402_1005Metric, F.Cu at (86.1, -56.1)
- added R36: 10k, Resistor_SMD:R_0402_1005Metric, F.Cu at (149.8, -66.4)
- added R37: 220k 1%, Resistor_SMD:R_0402_1005Metric, F.Cu at (155.0, -71.0)
- added R38: 69k8 1%, Resistor_SMD:R_0402_1005Metric, F.Cu at (137.0, -53.2)
- added R39: 10k, Resistor_SMD:R_0402_1005Metric, F.Cu at (130.1, -61.2)
- added R40: 220k 1%, Resistor_SMD:R_0402_1005Metric, F.Cu at (126.5, -42.0)
- added R41: 220k 1%, Resistor_SMD:R_0402_1005Metric, F.Cu at (133.0, -61.2)
- added R42: 75, Resistor_SMD:R_0402_1005Metric, F.Cu at (152.7, -82.7)
- added R43: 75, Resistor_SMD:R_0402_1005Metric, F.Cu at (161.4, -82.7)
- added R44: 75, Resistor_SMD:R_0402_1005Metric, F.Cu at (152.7, -80.8)
- added R45: 75, Resistor_SMD:R_0402_1005Metric, F.Cu at (149.8, -82.7)
- added R46: 75, Resistor_SMD:R_0402_1005Metric, F.Cu at (158.5, -82.7)
- added R47: 75, Resistor_SMD:R_0402_1005Metric, F.Cu at (161.4, -80.8)
- added R48: 75, Resistor_SMD:R_0402_1005Metric, F.Cu at (155.6, -80.8)
- added R49: 75, Resistor_SMD:R_0402_1005Metric, F.Cu at (187.2, -100.6)
- added R50: 75, Resistor_SMD:R_0402_1005Metric, F.Cu at (158.5, -80.8)
- added R51: 75, Resistor_SMD:R_0402_1005Metric, F.Cu at (149.8, -80.8)
- added R52: 75, Resistor_SMD:R_0402_1005Metric, F.Cu at (155.6, -82.7)
- added R53: 75, Resistor_SMD:R_0402_1005Metric, F.Cu at (164.3, -82.7)
- added R54: 75, Resistor_SMD:R_0402_1005Metric, F.Cu at (203.6, -113.7)
- added R55: 75, Resistor_SMD:R_0402_1005Metric, F.Cu at (190.1, -100.6)
- added R56: 1k5, Resistor_SMD:R_0402_1005Metric, F.Cu at (105.2, -99.6)
- added R57: 1k, Resistor_SMD:R_0402_1005Metric, F.Cu at (117.0, -111.6)
- added R58: 10k, Resistor_SMD:R_0402_1005Metric, F.Cu at (119.8, -113.6)
- added R59: 10k, Resistor_SMD:R_0402_1005Metric, F.Cu at (67.3, -36.6)
- added RJ1: DS1134-07-S8B0P, DS1134-07-S8B0P:RJ45-TH_DS1134-07-S8B0P, F.Cu at (129.3, 106.9)
- added RJ2: DS1134-07-S8B0P, DS1134-07-S8B0P:RJ45-TH_DS1134-07-S8B0P, F.Cu at (146.3, 106.9)
- added RJ3: DS1134-07-S8B0P, DS1134-07-S8B0P:RJ45-TH_DS1134-07-S8B0P, F.Cu at (129.3, 86.9)
- added RJ4: DS1134-07-S8B0P, DS1134-07-S8B0P:RJ45-TH_DS1134-07-S8B0P, F.Cu at (146.3, 86.9)
- added RJ5: DS1134-07-S8B0P, DS1134-07-S8B0P:RJ45-TH_DS1134-07-S8B0P, F.Cu at (129.3, 66.9)
- added TP10: TestPoint, TestPoint:TestPoint_Pad_1.5x1.5mm, F.Cu at (101.9, -98.9)
- added TP11: TestPoint, TestPoint:TestPoint_Pad_1.5x1.5mm, F.Cu at (131.1, -128.2)
- added TP12: TestPoint, TestPoint:TestPoint_Pad_1.5x1.5mm, F.Cu at (101.9, -106.0)
- added TP13: TestPoint, TestPoint:TestPoint_Pad_1.5x1.5mm, F.Cu at (73.8, -47.1)
- added TP14: TestPoint, TestPoint:TestPoint_Pad_1.5x1.5mm, F.Cu at (79.5, -52.3)
- added TP15: TestPoint, TestPoint:TestPoint_Pad_1.5x1.5mm, F.Cu at (63.7, -34.8)
- added TP16: TestPoint, TestPoint:TestPoint_Pad_1.5x1.5mm, F.Cu at (70.2, -43.4)
- added TP17: TestPoint, TestPoint:TestPoint_Pad_1.5x1.5mm, F.Cu at (87.6, -59.7)
- added TP18: TestPoint, TestPoint:TestPoint_Pad_1.5x1.5mm, F.Cu at (84.0, -58.9)
- added TP19: TestPoint, TestPoint:TestPoint_Pad_1.5x1.5mm, F.Cu at (97.6, -71.1)
- added TP20: TestPoint, TestPoint:TestPoint_Pad_1.5x1.5mm, F.Cu at (99.3, -74.6)
- added TP21: TestPoint, TestPoint:TestPoint_Pad_1.5x1.5mm, F.Cu at (76.0, -52.3)
- added TP22: TestPoint, TestPoint:TestPoint_Pad_1.5x1.5mm, F.Cu at (80.0, -56.3)
- added TP23: TestPoint, TestPoint:TestPoint_Pad_1.5x1.5mm, F.Cu at (70.2, -47.0)
- added TP24: TestPoint, TestPoint:TestPoint_Pad_1.5x1.5mm, F.Cu at (94.0, -70.2)
- added TP25: TestPoint, TestPoint:TestPoint_Pad_1.5x1.5mm, F.Cu at (94.9, -66.6)
- added TP26: TestPoint, TestPoint:TestPoint_Pad_1.5x1.5mm, F.Cu at (102.8, -74.6)
- added TP27: TestPoint, TestPoint:TestPoint_Pad_1.5x1.5mm, F.Cu at (91.3, -66.6)
- added TP28: TestPoint, TestPoint:TestPoint_Pad_1.5x1.5mm, F.Cu at (91.3, -63.1)
- added TP29: TestPoint, TestPoint:TestPoint_Pad_1.5x1.5mm, F.Cu at (64.1, -38.4)
- added TP30: TestPoint, TestPoint:TestPoint_Pad_1.5x1.5mm, F.Cu at (126.8, -44.7)
- added TP31: TestPoint, TestPoint:TestPoint_Pad_1.5x1.5mm, F.Cu at (137.3, -55.9)
- added TP32: TestPoint, TestPoint:TestPoint_Pad_1.5x1.5mm, F.Cu at (140.8, -55.9)
- added TP33: TestPoint, TestPoint:TestPoint_Pad_1.5x1.5mm, F.Cu at (142.2, -60.4)
- added TP8: TestPoint, TestPoint:TestPoint_Pad_1.5x1.5mm, F.Cu at (126.7, -122.9)
- added TP9: TestPoint, TestPoint:TestPoint_Pad_1.5x1.5mm, F.Cu at (105.5, -102.4)
- added U10: AP3402, Package_TO_SOT_SMD:TSOT-23-6, F.Cu at (146.0, -69.6)
- added U6: TPS2378DDAR, TPS2378DDAR:SO-8_L4.9-W3.9-P1.27-LS6.0-BL-EP, F.Cu at (61.3, -44.5)
- added U7: AP3402, Package_TO_SOT_SMD:TSOT-23-6, F.Cu at (154.0, -74.2)
- added U8: LM2576HVS-5, Package_TO_SOT_SMD:TO-263-5_TabPin3, F.Cu at (119.5, -52.7)
- added U9: MCP1703Ax-330xxTT, Package_TO_SOT_SMD:SOT-23, F.Cu at (138.0, -59.9)
- added Y1: 8MHz, Crystal:Crystal_SMD_5032-2Pin_5.0x3.2mm, F.Cu at (79.2, -84.9)
- added Y2: 25MHz 50ppm, Crystal:Crystal_SMD_3225-4Pin_3.2x2.5mm, F.Cu at (90.6, -74.2)
- C1: value 2u2 -> 100nF
- C10: value 4u7 -> 10u
- C11: value 1u -> 20pF
- C12: value 0u1 -> 20pF
- C13, C16, C17, C18, C20: value 0u1 -> 100nF
- C14, C22: value 10u -> 100nF
- C15, C21: value 0u1 -> 1uF
- C19: value 0u1 -> 2u2
- C2: value 2u2 -> 4u7
- C23, C24, C26: value 1uF -> 100nF
- C25: value 1uF -> 2u2
- C27: value 100n -> 22u
- C28: value 10u -> 22uF
- C4: value 100n -> 10u
- C5, C7, C8: value 100n -> 100nF
- C6: value 100n -> 1uF
- D1: value D_Schottky -> LED_GREEN; footprint Diode_SMD:D_SMA -> LED_SMD:LED_0603_1608Metric
- D10, D12, D14, D16, D18, D9: value LED GREEN -> LED_GREEN
- D11, D13, D15, D17, D19: value LED GREEN -> LED_YELLOW
- D2: value LED_ORANGE -> LED_YELLOW
- D3, D4: value LED GREEN -> 1N4148WS; footprint LED_SMD:LED_0603_1608Metric -> Diode_SMD:D_SOD-323
- D7: value LED GREEN -> LED_BLUE
- D8: value LED GREEN -> LED_RED
- J1: value Conn_02x03_Odd_Even -> TC2050-IDC-NL; footprint Connector_PinSocket_2.54mm:PinSocket_2x03_P2.54mm_Vertical -> Project:TAG-CONNECT_TC2050-IDC-NL
- J2: value Conn_02x03_Odd_Even -> Conn_02x17_Odd_Even; footprint Connector_PinSocket_2.54mm:PinSocket_2x03_P2.54mm_Vertical -> Connector_PinHeader_2.54mm:PinHeader_2x17_P2.54mm_Vertical
- J3, J6: value Conn_01x08 -> Conn_02x17_Odd_Even; footprint TerminalBlock_Phoenix:TerminalBlock_Phoenix_PT-1,5-8-3.5-H_1x08_P3.50mm_Horizontal -> Connector_PinHeader_2.54mm:PinHeader_2x17_P2.54mm_Vertical
- J4: value Conn_01x04 -> Conn_01x02; footprint TerminalBlock_Phoenix:TerminalBlock_Phoenix_PT-1,5-4-3.5-H_1x04_P3.50mm_Horizontal -> TerminalBlock_Phoenix:TerminalBlock_Phoenix_PT-1,5-2-3.5-H_1x02_P3.50mm_Horizontal
- J5: value Conn_01x03 -> Conn_01x02; footprint TerminalBlock_Phoenix:TerminalBlock_Phoenix_PT-1,5-3-3.5-H_1x03_P3.50mm_Horizontal -> TerminalBlock_Phoenix:TerminalBlock_Phoenix_PT-1,5-2-3.5-H_1x02_P3.50mm_Horizontal
- J7: value Conn_01x02 -> Conn_02x04_Odd_Even; footprint TerminalBlock_Phoenix:TerminalBlock_Phoenix_PT-1,5-2-3.5-H_1x02_P3.50mm_Horizontal -> Connector_PinHeader_2.54mm:PinHeader_2x04_P2.54mm_Vertical
- J8: value Conn_01x02 -> USB_C_Receptacle; footprint TerminalBlock_Phoenix:TerminalBlock_Phoenix_PT-1,5-2-3.5-H_1x02_P3.50mm_Horizontal -> Connector_USB:USB_C_Receptacle_Molex_105450-0101
- R10: value 49R9 -> 22
- R11, R12: value 49R9 -> 330
- R13, R14: value 2k2 -> 330
- R15: value 120 -> 6.04k 1%
- R16, R17, R18, R19, R21, R22, R24, R25, R26, R27, R6: value 220 -> 330
- R2: value 2K2 -> 120
- R20, R23, R28, R29, R30: value 220 -> 10k
- R3: value 1.5k -> 120
- R31: value 220 -> 30k
- R32: value 220 -> 24k9 1%
- R33: value 220 -> 22k
- R4: value 2K2 -> 47
- R7: value 220 -> 5k1
- R8: value 49R9 -> 5k1
- R9: value 4k87 -> 22
- SW1: value SW_DIP_x04 -> TS-1187A-B-A-B; footprint Button_Switch_SMD:SW_DIP_SPSTx04_Slide_Copal_CHS-04B_W7.62mm_P1.27mm -> TS-1187A-B-A-B:SW-SMD_4P-L5.1-W5.1-P3.70-LS6.5-TL-2
- TP1, TP2, TP3, TP4, TP5, TP6, TP7: footprint TestPoint:TestPoint_Pad_D2.0mm -> TestPoint:TestPoint_Pad_1.5x1.5mm
- U1: value STM32F407VGTx -> TJA1042T; footprint Package_QFP:LQFP-100_14x14mm_P0.5mm -> Package_SO:SOIC-8_3.9x4.9mm_P1.27mm
- U2: value MCP1703Ax-500xxTT -> MAX485E; footprint Package_TO_SOT_SMD:SOT-23 -> Package_SO:SOIC-8_3.9x4.9mm_P1.27mm
- U3: value DP83848KSQ_NOPB -> MAX485E; footprint Project:Texas_Instruments-DP83848KSQ_NOPB-0 -> Package_SO:SOIC-8_3.9x4.9mm_P1.27mm
- U4: value MCP1703Ax-330xxTT -> STM32H723ZGT6; footprint Package_TO_SOT_SMD:SOT-23 -> STM32H723ZGT6:LQFP-144_L20.0-W20.0-P0.50-LS22.0-BL
- U5: value MAX485E -> KSZ9896CTXC-TR; footprint Package_SO:SOIC-8_3.9x4.9mm_P1.27mm -> KSZ9896CTXC-TR:TQFP-128_L14.0-W14.0-P0.40-LS16.0-BL-EP
- moved C24 240.5 mm to (138.3, -131.6)
- moved D1 237.1 mm to (131.3, -131.3), turned to 0 degrees
- moved D9 236.4 mm to (122.9, -123.3), turned to 0 degrees
- moved D8 233.7 mm to (114.5, -116.9), turned to 0 degrees
- moved R13 227.9 mm to (114.0, -114.6)
- moved R14 227.2 mm to (121.6, -117.2)
- moved C3 227.0 mm to (141.2, -131.6), turned to 0 degrees
- moved R6 226.2 mm to (116.9, -113.6)
- moved C26 226.2 mm to (132.7, -123.5), turned to 0 degrees
- moved U3 225.5 mm to (117.1, -129.4)
- moved R5 224.7 mm to (134.3, -128.0)
- moved C1 223.4 mm to (134.3, -126.1), turned to 0 degrees
- moved J8 223.4 mm to (85.3, -102.8)
- moved J1 222.8 mm to (108.1, -128.1)
- moved R12 221.5 mm to (130.7, -125.4), turned to 0 degrees
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Connections:
- C1 pad 1: GND -> +3V3
- C1 pad 2: Net-(C1-Pad2) -> GND
- C10 pad 1: +3V3 -> +5V
- C11 pad 1: +3V3 -> Net-(C11-Pad1)
- C12 pad 1: +3V3 -> Net-(C12-Pad1)
- C15 pad 1: +3V3 -> Net-(C15-Pad1)
- C16 pad 1: +3V3 -> Net-(C15-Pad1)
- C17 pad 1: GND -> +3V3
- C17 pad 2: +3V3 -> GND
- C18 pad 1: Net-(C18-Pad1) -> +3V3
- C2 pad 1: Net-(C2-Pad1) -> GND
- C2 pad 2: GND -> +3V3
- C21 pad 1: Net-(C21-Pad1) -> GND
- C21 pad 2: GND -> +3V3
- C22 pad 1: Net-(C21-Pad1) -> +3V3
- C23 pad 1: +5V -> +3V3
- C24 pad 1: /12V_D -> +3V3
- C25 pad 1: +5V -> Net-(C25-Pad1)
- C26 pad 1: +3V3 -> GND
- C26 pad 2: GND -> +3V3
- C27 pad 1: +5V -> GND
- C27 pad 2: GND -> +2V5
- C28 pad 1: +5V -> GND
- C28 pad 2: GND -> +1V2
- C3 pad 1: +3V3 -> +5V
- C4 pad 1: +3V3 -> +5V
- C5 pad 1: +3V3 -> GND
- C5 pad 2: GND -> +3V3
- C6 pad 1: +3V3 -> GND
- C6 pad 2: GND -> +3V3
- C9 pad 1: +3V3 -> +5V
- D1 pad 1: /12V_D -> /LED_GREEN
- D1 pad 2: +12V -> Net-(D1-Pad2)
- D12 pad 1: GND -> Net-(D12-Pad1)
- D13 pad 1: GND -> Net-(D13-Pad1)
- D14 pad 1: GND -> Net-(D14-Pad1)
- D15 pad 1: GND -> Net-(D15-Pad1)
- D16 pad 1: GND -> Net-(D16-Pad1)
- D17 pad 1: GND -> Net-(D17-Pad1)
- D18 pad 1: GND -> Net-(D18-Pad1)
- D19 pad 1: GND -> Net-(D19-Pad1)
- D2 pad 1: /STATUS_LED -> /LED_YELLOW
- D3 pad 1: GND -> +3V3
- D3 pad 2: Net-(D3-Pad2) -> Net-(C49-Pad1)
- D4 pad 1: Net-(D4-Pad1) -> /~{ETH_RESET}
- D4 pad 2: Net-(D4-Pad2) -> Net-(C49-Pad1)
- D7 pad 1: Net-(D7-Pad1) -> /LED_BLUE
- D8 pad 1: Net-(D8-Pad1) -> /LED_RED
- D9 pad 1: Net-(D9-Pad1) -> GND
- J1 pad 1: /PWM_OUT_2 -> /NRST
- J1 pad 2: /PWM_OUT_1 -> /DBG_SWDIO
- J1 pad 3: +5V -> GND
- J1 pad 4: +5V -> GND
- J1 pad 5: GND -> unconnected-(J1-Pad5)
- J1 pad 6: GND -> /DBG_SWCLK
- J2 pad 1: /PWM_OUT_4 -> +5V
- J2 pad 2: /PWM_OUT_3 -> GND
- J2 pad 3: +5V -> /I2C1_SCL
- J2 pad 4: +5V -> /SPI1_CS
- J2 pad 5: GND -> /I2C1_SDA
- J2 pad 6: GND -> /SPI1_SCLK
- J3 pad 1: /Digital IO/DIN_1 -> +5V
- J3 pad 2: /Digital IO/DIN_2 -> GND
- J3 pad 3: /Digital IO/DIN_3 -> /DIO1
- J3 pad 4: /Digital IO/DIN_4 -> /DIO15
- J3 pad 5: /Digital IO/DIN_5 -> /DIO2
- J3 pad 6: /Digital IO/DIN_6 -> /DIO16
- J3 pad 7: /Digital IO/DIN_7 -> /DIO3
- J3 pad 8: /Digital IO/DIN_8 -> GND
- J4 pad 1: /AIN_1 -> /CANH
- J4 pad 2: /AIN_2 -> /CANL
- J5 pad 1: /PWM_IN_1 -> VIN
- J5 pad 2: /PWM_IN_2 -> GND
- J6 pad 1: /Digital IO/DOUT_1 -> +5V
- J6 pad 2: /Digital IO/DOUT_2 -> GND
- J6 pad 3: /Digital IO/DOUT_3 -> /PWM1
- J6 pad 4: /Digital IO/DOUT_4 -> /QE1_A
- J6 pad 5: /Digital IO/DOUT_5 -> /PWM2
- J6 pad 6: /Digital IO/DOUT_6 -> /QE1_B
- J6 pad 7: /Digital IO/DOUT_7 -> /PWM3
- J6 pad 8: /Digital IO/DOUT_8 -> /QE1_I
- J7 pad 1: /AOUT_1 -> VDC
- J7 pad 2: /AOUT_2 -> VDC
- JP1 pad 1: Net-(J12-Pad7) -> Net-(J1-Pad7)
- R1 pad 1: GND -> unconnected-(R1-Pad1)
- R1 pad 2: Net-(R1-Pad2) -> unconnected-(R1-Pad2)
- R10 pad 1: /ethernet/TD- -> /USB_D+
- R10 pad 2: +3V3 -> /D+
- R11 pad 1: /ethernet/RD+ -> +3V3
- R11 pad 2: +3V3 -> Net-(D2-Pad2)
- R12 pad 1: /ethernet/RD- -> +3V3
- R12 pad 2: +3V3 -> Net-(D7-Pad2)
- R13 pad 1: /ethernet/LED_SPEED -> +3V3
- R13 pad 2: +3V3 -> Net-(D8-Pad2)
- R14 pad 2: /ethernet/LED_LINK -> Net-(D9-Pad2)
- R15 pad 1: /DMX/DMX- -> Net-(R15-Pad1)
- R15 pad 2: /DMX/DMX+ -> GND
- R16 pad 2: Net-(D2-Pad2) -> Net-(D10-Pad2)
- R17 pad 2: Net-(D3-Pad2) -> Net-(D11-Pad2)
- R18 pad 2: Net-(D4-Pad2) -> Net-(D12-Pad2)
- R19 pad 2: Net-(D5-Pad2) -> Net-(D13-Pad2)
- R2 pad 1: Net-(R2-Pad1) -> /RS485_1_B
- R2 pad 2: +3V3 -> /RS485_1_A
- R20 pad 1: +3V3 -> /~{ETH_INTERRUPT}
- R20 pad 2: Net-(D6-Pad2) -> +3V3
- R21 pad 2: Net-(D7-Pad2) -> Net-(D14-Pad2)
- R22 pad 2: Net-(D8-Pad2) -> Net-(D15-Pad2)
- R23 pad 1: +3V3 -> /~{ETH_PME}
- R23 pad 2: Net-(D9-Pad2) -> +3V3
- R24 pad 2: Net-(D10-Pad2) -> Net-(D16-Pad2)
- R25 pad 2: Net-(D11-Pad2) -> Net-(D17-Pad2)
- R26 pad 1: /Digital IO/DOUT_1 -> +3V3
- R26 pad 2: Net-(D12-Pad2) -> Net-(D18-Pad2)
- R27 pad 1: /Digital IO/DOUT_2 -> +3V3
- R27 pad 2: Net-(D13-Pad2) -> Net-(D19-Pad2)
- R28 pad 1: /Digital IO/DOUT_3 -> /ETH_RXD0
- R28 pad 2: Net-(D14-Pad2) -> +3V3
- R29 pad 1: /Digital IO/DOUT_4 -> Net-(R29-Pad1)
- R29 pad 2: Net-(D15-Pad2) -> +3V3
- R3 pad 1: /ETH_MDIO -> /RS485_2_B
- R3 pad 2: +3V3 -> /RS485_2_A
- R30 pad 1: /Digital IO/DOUT_5 -> Net-(R30-Pad1)
- R30 pad 2: Net-(D16-Pad2) -> GND
- R31 pad 1: /Digital IO/DOUT_6 -> VIN
- R31 pad 2: Net-(D17-Pad2) -> Net-(R31-Pad2)
- R32 pad 1: /Digital IO/DOUT_7 -> Net-(R32-Pad1)
- R32 pad 2: Net-(D18-Pad2) -> VDC
- R33 pad 1: /Digital IO/DOUT_8 -> Net-(R33-Pad1)
- R33 pad 2: Net-(D19-Pad2) -> Net-(D22-Pad1)
- R4 pad 1: /ETH_CRS_DV -> Net-(R4-Pad1)
- R4 pad 2: +3V3 -> Net-(C15-Pad1)
- R5 pad 1: Net-(R5-Pad1) -> /Power Management/~{EN}
- R5 pad 2: +3V3 -> GND
- R6 pad 2: Net-(J11-PadL4) -> Net-(D1-Pad2)
- R7 pad 1: +3V3 -> GND
- R7 pad 2: Net-(J11-PadL1) -> Net-(J8-PadA5)
- R8 pad 1: /ethernet/TD+ -> Net-(J8-PadB5)
- R8 pad 2: +3V3 -> GND
- R9 pad 1: Net-(R9-Pad1) -> /USB_D-
- R9 pad 2: GND -> /D-
- SW1 pad 1: GND -> unconnected-(SW1-Pad1)
- SW1 pad 2: GND -> Net-(R57-Pad1)
- SW1 pad 3: GND -> unconnected-(SW1-Pad3)
- TP1 pad 1: /DMX_RX -> /ETH_SPI_SCLK
- TP2 pad 1: /DMX_TX_EN -> /ETH_SPI_CS
- TP3 pad 1: /DMX_TX -> /ETH_SPI_MISO
- TP4 pad 1: Net-(R1-Pad2) -> /ETH_SPI_MOSI
- TP5 pad 1: /NRST -> Net-(TP5-Pad1)
- TP6 pad 1: /SWDIO -> /ethernet/~{CDB}
- TP7 pad 1: /SWCLK -> /NRST
- U1 pad 1: unconnected-(U1-Pad1) -> /CAN_TX
- U1 pad 2: unconnected-(U1-Pad2) -> GND
- U1 pad 3: unconnected-(U1-Pad3) -> +5V
- U1 pad 4: /PWM_IN_1 -> /CAN_RX
- U1 pad 6: +3V3 -> /CANL
- U1 pad 7: unconnected-(U1-Pad7) -> /CANH
- U1 pad 8: unconnected-(U1-Pad8) -> GND
- U2 pad 1: GND -> /RS485_1_RX
- U2 pad 2: +5V -> /RS485_1_DE
- U2 pad 3: /12V_D -> /RS485_1_DE
- U3 pad 1: +3V3 -> /RS485_2_RX
- U3 pad 2: unconnected-(U3-Pad2) -> /RS485_2_DE
- U3 pad 3: /ETH_TX_EN -> /RS485_2_DE
- U3 pad 4: /ETH_TXD0 -> /RS485_2_TX
- U3 pad 5: /ETH_TXD1 -> GND
- U3 pad 6: unconnected-(U3-Pad6) -> /RS485_2_A
- U3 pad 7: unconnected-(U3-Pad7) -> /RS485_2_B
- U3 pad 8: unconnected-(U3-Pad8) -> +5V
- U4 pad 1: GND -> /ETH_SPI_SCLK
- U4 pad 2: +3V3 -> unconnected-(U4-Pad2)
- U4 pad 3: +5V -> /ETH_SPI_CS
- U5 pad 1: /DMX_RX -> /ethernet/IETH1A+
- U5 pad 2: /DMX_TX_EN -> /ethernet/IETH1A-
- U5 pad 3: /DMX_TX_EN -> +1V2
- U5 pad 4: /DMX_TX -> /ethernet/IETH1B+
- U5 pad 5: GND -> /ethernet/IETH1B-
- U5 pad 6: /DMX/DMX+ -> /ethernet/IETH1C+
- U5 pad 7: /DMX/DMX- -> /ethernet/IETH1C-
- U5 pad 8: +5V -> /ethernet/IETH1D+
Routing:
- net +3V3: track 317.2 -> 0.00 mm, vias 19 -> 0
- net +5V: track 134.6 -> 0.00 mm, vias 3 -> 0
- net /AIN_4: track 66.7 -> 0.00 mm, vias 1 -> 0
- net /AIN_3: track 62.5 -> 0.00 mm, vias 1 -> 0
- net /AOUT_1: track 54.9 -> 0.00 mm, vias 2 -> 0
- net /ETH_TXD1: track 54.6 -> 0.00 mm, vias 2 -> 0
- net /AOUT_2: track 52.9 -> 0.00 mm, vias 1 -> 0
- net /ETH_TXD0: track 52.7 -> 0.00 mm, vias 2 -> 0
- net /NRST: track 52.1 -> 0.00 mm, vias 2 -> 0
- net /AIN_2: track 49.3 -> 0.00 mm, vias 1 -> 0
- net /PWM_IN_1: track 47.8 -> 0.00 mm, vias 1 -> 0
- net /ethernet/LED_LINK: track 47.1 -> 0.00 mm, vias 2 -> 0
- net /AIN_1: track 46.2 -> 0.00 mm, vias 1 -> 0
- net /Digital IO/DIN_8: track 45.7 -> 0.00 mm
- net /SWDIO: track 44.5 -> 0.00 mm, vias 2 -> 0
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Other:
- board size 100 x 70 mm -> 125 x 75 mm
- board text removed: "+5V"
- board text removed: "+V"
- board text removed: "1"
- board text removed: "2"
- board text removed: "3"
- board text removed: "4"
- board text removed: "A"
- board text removed: "B"
- board text removed: "C"
- board text removed: "D"
- board text removed: "DMX OUT"
- board text removed: "GND"
- board text removed: "JMS"
- board text removed: "MODE SEL"
- board text removed: "REV 2"
- board text removed: "UNIFIED FIELD ELECTRONICS"
