File: electronics/hardware/jms_ufe_controller/jms_ufe_controller.kicad_sch (KiCad schematic)
At the start: 60 parts, among them J1 Conn_02x03_Odd_Even, J12 TC2050-IDC-NL, J2 Conn_02x03_Odd_Even, J3 Conn_01x04, J4 Conn_01x04, J5 Conn_01x03, J6 Conn_01x04, J7 Conn_01x02, J8 Conn_01x02, J9 Conn_01x04, SW1 SW_DIP_x04, U1 STM32F407VGTx, U2 MCP1703Ax-500xxTT, U4 MCP1703Ax-330xxTT

Commit message: UFE Rev 2 off to the board fab
Parts:
- removed D10, D11, D4, D5, D6, D7, D8, D9: LED GREEN, LED_SMD:LED_0603_1608Metric, symbol Device:LED
- removed J3, J6: Conn_01x04, TerminalBlock_Phoenix:TerminalBlock_Phoenix_PT-1,5-4-5.0-H_1x04_P5.00mm_Horizontal, symbol Connector_Generic:Conn_01x04
- removed R18, R19, R20, R21, R22, R23, R24, R25: 220, Resistor_SMD:R_0402_1005Metric, symbol Device:R_US
- J4, J9: footprint TerminalBlock_Phoenix:TerminalBlock_Phoenix_PT-1,5-4-5.0-H_1x04_P5.00mm_Horizontal -> TerminalBlock_Phoenix:TerminalBlock_Phoenix_PT-1,5-4-3.5-H_1x04_P3.50mm_Horizontal
- J5: footprint TerminalBlock_Phoenix:TerminalBlock_Phoenix_PT-1,5-3-5.0-H_1x03_P5.00mm_Horizontal -> TerminalBlock_Phoenix:TerminalBlock_Phoenix_PT-1,5-3-3.5-H_1x03_P3.50mm_Horizontal
- J7, J8: footprint TerminalBlock_Phoenix:TerminalBlock_Phoenix_PT-1,5-2-5.0-H_1x02_P5.00mm_Horizontal -> TerminalBlock_Phoenix:TerminalBlock_Phoenix_PT-1,5-2-3.5-H_1x02_P3.50mm_Horizontal
- U1: LCSC (none) -> C12345
Connections:
- net Digital IO/DOUT_5: now reaches U1.85 (PD4)
- net Digital IO/DOUT_6: now reaches U1.86 (PD5)
- net Digital IO/DOUT_7: now reaches U1.87 (PD6)
- net Digital IO/DOUT_8: now reaches U1.88 (PD7)
- net DIN1_LED renamed Digital IO/DIN_2
- net DIN2_LED renamed Digital IO/DIN_4
- net DIN3_LED renamed Digital IO/DIN_6
- net DIN4_LED renamed Digital IO/DIN_8
- net DIN_1 renamed Digital IO/DIN_1
- net DIN_2 renamed Digital IO/DIN_3
- net DIN_3 renamed Digital IO/DIN_5
- net DIN_4 renamed Digital IO/DIN_7
- net DOUT_1 renamed Digital IO/DOUT_1
- net DOUT_2 renamed Digital IO/DOUT_2
- net DOUT_3 renamed Digital IO/DOUT_3
- net DOUT_4 renamed Digital IO/DOUT_4
Other:
- added sheet Digital IO (digital.kicad_sch)
- moved on the sheet: C1, C10, C11, C2, C23, C24, C25, C26, C3, C4, C5, C6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

Commit message: UFE Rev 3 - first try
Parts:
- removed D1: D_Schottky, Diode_SMD:D_SMA, symbol Device:D_Schottky
- removed D2: LED_ORANGE, LED_SMD:LED_0603_1608Metric, symbol Device:LED
- removed D3: LED GREEN, LED_SMD:LED_0603_1608Metric, symbol Device:LED
- removed J1, J2: Conn_02x03_Odd_Even, Connector_PinSocket_2.54mm:PinSocket_2x03_P2.54mm_Vertical, symbol Connector_Generic:Conn_02x03_Odd_Even
- removed J4, J9: Conn_01x04, TerminalBlock_Phoenix:TerminalBlock_Phoenix_PT-1,5-4-3.5-H_1x04_P3.50mm_Horizontal, symbol Connector_Generic:Conn_01x04
- removed J5: Conn_01x03, TerminalBlock_Phoenix:TerminalBlock_Phoenix_PT-1,5-3-3.5-H_1x03_P3.50mm_Horizontal, symbol Connector_Generic:Conn_01x03
- removed J7, J8: Conn_01x02, TerminalBlock_Phoenix:TerminalBlock_Phoenix_PT-1,5-2-3.5-H_1x02_P3.50mm_Horizontal, symbol Connector_Generic:Conn_01x02
- removed R1: 10k, Resistor_SMD:R_0402_1005Metric, symbol Device:R_US
- removed R17: 220, Resistor_SMD:R_0402_1005Metric, symbol Device:R_US
- removed SW1: SW_DIP_x04, Button_Switch_SMD:SW_DIP_SPSTx04_Slide_Copal_CHS-04B_W7.62mm_P1.27mm, symbol Switch:SW_DIP_x04
- removed U1: STM32F407VGTx, Package_QFP:LQFP-100_14x14mm_P0.5mm, symbol MCU_ST_STM32F4:STM32F407VGTx
- removed U2: MCP1703Ax-500xxTT, Package_TO_SOT_SMD:SOT-23, symbol Regulator_Linear:MCP1703Ax-500xxTT
- removed U4: MCP1703Ax-330xxTT, Package_TO_SOT_SMD:SOT-23, symbol Regulator_Linear:MCP1703Ax-330xxTT
- added C12: 20pF, Capacitor_SMD:C_0402_1005Metric, symbol Device:C_Small
- added C13, C14, C16, C17, C18, C20, C22: 100nF, Capacitor_SMD:C_0402_1005Metric, symbol Device:C_Small
- added C15, C21, C98: 1uF, Capacitor_SMD:C_0402_1005Metric, symbol Device:C_Small
- added C19: 2u2, Capacitor_SMD:C_0402_1005Metric, symbol Device:C_Small
- added D1, D9: LED_GREEN, LED_SMD:LED_0603_1608Metric, symbol Device:LED_Small
- added D2: LED_YELLOW, LED_SMD:LED_0603_1608Metric, symbol Device:LED_Small
- added D7: LED_BLUE, LED_SMD:LED_0603_1608Metric, symbol Device:LED_Small
- added D8: LED_RED, LED_SMD:LED_0603_1608Metric, symbol Device:LED_Small
- added J2, J3, J6: Conn_02x17_Odd_Even, Connector_PinHeader_2.54mm:PinHeader_2x17_P2.54mm_Vertical, symbol Connector_Generic:Conn_02x17_Odd_Even
- added J4, J5: Conn_01x02, TerminalBlock_Phoenix:TerminalBlock_Phoenix_PT-1,5-2-3.5-H_1x02_P3.50mm_Horizontal, symbol Connector_Generic:Conn_01x02
- added J8: USB_C_Receptacle, Connector_USB:USB_C_Receptacle_Molex_105450-0101, symbol Connector:USB_C_Receptacle
- added R1, R5, R58: 10k, Resistor_SMD:R_0402_1005Metric, symbol Device:R_Small
- added R10, R9: 22, Resistor_SMD:R_0402_1005Metric, symbol Device:R_US
- added R11, R12, R13, R14: 330, Resistor_SMD:R_0402_1005Metric, symbol Device:R_Small
- added R2, R3: 120, Resistor_SMD:R_0402_1005Metric, symbol Device:R_Small
- added R4: 47, Resistor_SMD:R_0402_1005Metric, symbol Device:R_Small
- added R56: 1k5, Resistor_SMD:R_0402_1005Metric, symbol Device:R_US
- added R57: 1k, Resistor_SMD:R_0402_1005Metric, symbol Device:R_Small
- added R7, R8: 5k1, Resistor_SMD:R_0402_1005Metric, symbol Device:R_US
- added SW1: TS-1187A-B-A-B, TS-1187A-B-A-B:SW-SMD_4P-L5.1-W5.1-P3.70-LS6.5-TL-2, symbol TS-1187A-B-A-B:TS-1187A-B-A-B
- added TP1, TP10, TP11, TP12, TP2, TP3, TP8, TP9: TestPoint, TestPoint:TestPoint_Pad_1.5x1.5mm, symbol Connector:TestPoint
- added U1: TJA1042T, Package_SO:SOIC-8_3.9x4.9mm_P1.27mm, symbol Interface_CAN_LIN:TJA1042T
- added U2, U3: MAX485E, Package_SO:SOIC-8_3.9x4.9mm_P1.27mm, symbol Interface_UART:MAX485E
- added U4: STM32H723ZGT6, STM32H723ZGT6:LQFP-144_L20.0-W20.0-P0.50-LS22.0-BL, symbol STM32H723ZGT6:STM32H723ZGT6
- added Y1: 8MHz, Crystal:Crystal_SMD_5032-2Pin_5.0x3.2mm, symbol Device:Crystal_Small
- C1: value 2u2 -> 100nF
- C10: value 4u7 -> 10u
- C11: value 1u -> 20pF
- C2: value 2u2 -> 4u7
- C23, C24, C26: value 1uF -> 100nF
- C25: value 1uF -> 2u2
- C4: value 100n -> 10u
- C5, C7, C8: value 100n -> 100nF
- C6: value 100n -> 1uF
- R6: renamed from R16; value 220 -> 330; symbol Device:R_US -> Device:R_Small
- TP4, TP5, TP6, TP7: footprint TestPoint:TestPoint_Pad_D2.0mm -> TestPoint:TestPoint_Pad_1.5x1.5mm
- renumbered H2 to H1, H3 to H2, H1 to H3, J12 to J1
Connections:
- net 12V_D is gone; now on net +3V3: C24.1
- net +3V3: now also C1.1, C2.2, C23.1, C26.2, C5.2, C6.2, C13.1, C14.1, C17.1, C18.1, C20.2, C21.2, C22.1, J2.31 (Pin_31), J2.33 (Pin_33), J3.33 (Pin_33), J6.27 (Pin_27), J6.29 (Pin_29), J6.31 (Pin_31), J6.33 (Pin_33), R11.1, R12.1, R13.1, R14.1, R56.2, R58.2, U4.108 (VDD), U4.121 (VDD), U4.131 (VDD), U4.143 (PDR_ON), U4.144 (VDD), U4.17 (VDD), U4.30 (VDD), U4.39 (VDD), U4.52 (VDD), U4.6 (VBAT), U4.62 (VDD), U4.72 (VDD), U4.84 (VDD), U4.95 (VDD33USB); no longer C10.1, C11.1, C26.1, C3.1, C4.1, C5.1, C6.1, C9.1
- net +5V: now also C10.1, C3.1, C4.1, C9.1, J2.1 (Pin_1), J3.1 (Pin_1), J6.1 (Pin_1), U1.3 (VCC), U2.8 (VCC), U3.8 (VCC); no longer C23.1, C25.1
- net ETH_CRS_DV: now also U4.43 (PA7)
- net ETH_MDC: now also TP8.1, U4.27 (PC1)
- net ETH_MDIO: now also TP9.1, U4.36 (PA2)
- net ETH_RXD0: now also U4.44 (PC4)
- net ETH_RXD1: now also U4.45 (PC5)
- net ETH_TXD0: now also U4.73 (PB12)
- net ETH_TXD1: now also U4.74 (PB13)
- net ETH_TX_EN: now also U4.70 (PB11)
- net GND: now also C1.2, C2.1, C26.1, C5.1, C6.1, C12.2, C13.2, C14.2, C15.2, C16.2, C17.2, C18.2, C19.2, C20.1, C21.1, C22.2, C98.2, D9.1 (K), J2.19 (Pin_19), J2.2 (Pin_2), J2.20 (Pin_20), J2.21 (Pin_21), J2.30 (Pin_30), J2.32 (Pin_32), J2.34 (Pin_34), J3.17 (Pin_17), J3.2 (Pin_2), J3.34 (Pin_34), J3.8 (Pin_8), J5.2 (Pin_2), J6.10 (Pin_10), J6.17 (Pin_17), J6.18 (Pin_18), J6.2 (Pin_2), J6.23 (Pin_23), J6.25 (Pin_25), J6.26 (Pin_26), J6.34 (Pin_34), J6.9 (Pin_9), J8.A1 (GND), J8.A12 (GND), J8.B1 (GND), J8.B12 (GND), J8.S1 (SHIELD), R5.2, R7.1, R8.2, SW1.4 (D), U1.2 (GND), U1.8 (STB), U2.5 (GND), U3.5 (GND), U4.107 (VSS), U4.120 (VSS), U4.130 (VSS), U4.16 (VSS), U4.31 (VSSA), U4.38 (VSS), U4.51 (VSS), U4.61 (VSS), U4.83 (VSS), U4.94 (VSS); no longer C1.1, C2.2, C26.2, C5.2, C6.2
- net NRST: now also TP7.1, U4.25 (NRST); no longer TP5.1
- net ETH_SPI_MOSI: now reaches TP4.1
- net ETH_SPI_MOSI: now also U4.5 (PE6)
- net at R6.2: now also D1.2 (A)
- net SWCLK renamed DBG_SWCLK
- net DBG_SWCLK: now also U4.109 (PA14); no longer TP7.1
- net SWDIO renamed DBG_SWDIO
- net DBG_SWDIO: now also U4.105 (PA13); no longer TP6.1
- new net: R4.1, U4.32 (VREF+)
- new net: C15.1, C16.1, R4.2, U4.33 (VDDA)
- new net: C12.1, U4.24 (PH1-OSC_OUT), Y1.1
- new net: J8.A5 (CC1), R7.2
- new net: J8.B5 (CC2), R8.1
- new net: D7.2 (A), R12.2
- new net: D2.2 (A), R11.2
- new net: C19.1, U4.106 (VCAP)
- new net: D8.2 (A), R13.2
- new net: C25.1, U4.71 (VCAP)
- new net: TP5.1, U4.138 (BOOT0)
- new net: C11.1, U4.23 (PH0-OSC_IN), Y1.2
- new net: J8.A4 (VBUS), J8.A9 (VBUS), J8.B4 (VBUS), J8.B9 (VBUS)
- new net: D9.2 (A), R14.2
- new net: R57.1, SW1.2 (B)
- new net AI1: J3.14 (Pin_14), U4.29 (PC3_C)
- new net AI10: J3.32 (Pin_32), U4.13 (PF3)
- new net AI2: J3.16 (Pin_16), U4.28 (PC2_C)
- new net AI3: J3.18 (Pin_18), U4.22 (PF10)
- new net AI4: J3.20 (Pin_20), U4.21 (PF9)
- new net AI5: J3.22 (Pin_22), U4.20 (PF8)
- new net AI6: J3.24 (Pin_24), U4.19 (PF7)
- new net AI7: J3.26 (Pin_26), U4.18 (PF6)
- new net AI8: J3.28 (Pin_28), U4.15 (PF5)
- new net AI9: J3.30 (Pin_30), U4.14 (PF4)
- new net AO1: J3.10 (Pin_10), U4.40 (PA4)
- new net AO2: J3.12 (Pin_12), U4.41 (PA5)
- new net CANH: J4.1 (Pin_1), U1.7 (CANH)
- new net CANL: J4.2 (Pin_2), U1.6 (CANL)
- new net CAN_RX: U1.4 (RXD), U4.135 (PB5)
- new net CAN_TX: U1.1 (TXD), U4.136 (PB6)
- new net D+: J8.A6 (D+), J8.B6 (D+), R10.2
- new net D-: J8.A7 (D-), J8.B7 (D-), R9.2
- new net DBG_UART_RX: TP12.1, U4.85 (PD14)
- new net DBG_UART_TX: TP11.1, U4.86 (PD15)
- new net DIO1: J3.3 (Pin_3), U4.12 (PF2)
- new net DIO10: J3.23 (Pin_23), U4.87 (PG2)
- new net DIO11: J3.25 (Pin_25), U4.88 (PG3)
- new net DIO12: J3.27 (Pin_27), U4.89 (PG4)
- new net DIO13: J3.29 (Pin_29), U4.90 (PG5)
- new net DIO14: J3.31 (Pin_31), U4.91 (PG6)
- new net DIO15: J3.4 (Pin_4), U4.92 (PG7)
- new net DIO16: J3.6 (Pin_6), U4.98 (PC8)
- new net DIO2: J3.5 (Pin_5), U4.26 (PC0)
- new net DIO3: J3.7 (Pin_7), U4.53 (PF13)
- new net DIO4: J3.9 (Pin_9), U4.63 (PE10)
- new net DIO5: J3.11 (Pin_11), U4.65 (PE12)
- new net DIO6: J3.13 (Pin_13), U4.68 (PE15)
- new net DIO7: J3.15 (Pin_15), U4.76 (PB15)
- new net DIO8: J3.19 (Pin_19), U4.79 (PD10)
- new net DIO9: J3.21 (Pin_21), U4.80 (PD11)
- new net ETH_REF_CLK: U4.35 (PA1)
- new net ETH_SPI_CS: TP2.1, U4.3 (PE4)
- new net ETH_SPI_MISO: TP3.1, U4.4 (PE5)
- new net ETH_SPI_SCLK: TP1.1, U4.1 (PE2)
- new net FACTORY_RESET_SW: C98.1, R57.2, R58.1, U4.56 (PG0)
- new net I2C1_SCL: J2.3 (Pin_3), U4.139 (PB8)
- new net I2C1_SDA: J2.5 (Pin_5), U4.140 (PB9)
- new net I2C2_SCL: J2.7 (Pin_7), U4.11 (PF1)
- new net I2C2_SDA: J2.9 (Pin_9), U4.10 (PF0)
- new net I2C3_SCL: J2.11 (Pin_11), U4.100 (PA8)
- new net I2C3_SDA: J2.13 (Pin_13), U4.99 (PC9)
- new net I2C4_SCL: J2.15 (Pin_15), U4.54 (PF14)
- new net I2C4_SDA: J2.17 (Pin_17), U4.55 (PF15)
- new net LED_BLUE: D7.1 (K), U4.47 (PB1)
- new net LED_GREEN: D1.1 (K), U4.42 (PA6)
- new net LED_RED: D8.1 (K), U4.48 (PB2)
- new net LED_YELLOW: D2.1 (K), U4.46 (PB0)
- new net PWM1: J6.3 (Pin_3), U4.60 (PE9)
- new net PWM2: J6.5 (Pin_5), U4.64 (PE11)
- new net PWM3: J6.7 (Pin_7), U4.66 (PE13)
- new net PWM4: J6.11 (Pin_11), U4.67 (PE14)
- new net PWM5: J6.13 (Pin_13), U4.34 (PA0)
- new net PWM6: J6.15 (Pin_15), U4.133 (PB3)
- new net PWM7: J6.19 (Pin_19), U4.69 (PB10)
- new net PWM8: J6.21 (Pin_21), U4.37 (PA3)
- new net Power Management/~{EN}: R5.1, TP10.1
- new net QE1_A: J6.4 (Pin_4), U4.96 (PC6)
- new net QE1_B: J6.6 (Pin_6), U4.97 (PC7)
- new net QE1_I: J6.8 (Pin_8), U4.114 (PD0)
- new net QE2_A: J6.12 (Pin_12), U4.81 (PD12)
- new net QE2_B: J6.14 (Pin_14), U4.82 (PD13)
- new net QE2_I: J6.16 (Pin_16), U4.115 (PD1)
- new net QE3_A: J6.20 (Pin_20), U4.127 (PG12)
- new net QE3_B: J6.22 (Pin_22), U4.128 (PG13)
- new net QE3_I: J6.24 (Pin_24), U4.116 (PD2)
- new net QE4_A: J6.28 (Pin_28), U4.49 (PF11)
- new net QE4_B: J6.30 (Pin_30), U4.50 (PF12)
- new net QE4_I: J6.32 (Pin_32), U4.117 (PD3)
- new net RS485_1_A: J2.22 (Pin_22), R2.2, U2.6 (A)
- new net RS485_1_B: J2.24 (Pin_24), R2.1, U2.7 (B)
- new net RS485_1_DE: U2.2 (~{RE}), U2.3 (DE), U4.75 (PB14)
- new net RS485_1_RX: U2.1 (RO), U4.78 (PD9)
- new net RS485_1_TX: U2.4 (DI), U4.77 (PD8)
- new net RS485_2_A: J2.26 (Pin_26), R3.2, U3.6 (A)
- new net RS485_2_B: J2.28 (Pin_28), R3.1, U3.7 (B)
- new net RS485_2_DE: U3.2 (~{RE}), U3.3 (DE), U4.110 (PA15)
- new net RS485_2_RX: U3.1 (RO), U4.112 (PC11)
- new net RS485_2_TX: U3.4 (DI), U4.111 (PC10)
- new net SPI1_CS: J2.4 (Pin_4), U4.125 (PG10)
- new net SPI1_MISO: J2.8 (Pin_8), U4.124 (PG9)
- new net SPI1_MOSI: J2.10 (Pin_10), U4.123 (PD7)
- new net SPI1_SCLK: J2.6 (Pin_6), U4.126 (PG11)
- new net SPI6_CS: J2.12 (Pin_12), U4.93 (PG8)
- new net SPI6_MISO: J2.16 (Pin_16), U4.134 (PB4)
- new net SPI6_MOSI: J2.18 (Pin_18), U4.129 (PG14)
- new net SPI6_SCLK: J2.14 (Pin_14), U4.113 (PC12)
- new net UART1_RX: J2.23 (Pin_23), U4.102 (PA10)
- new net UART1_TX: J2.25 (Pin_25), U4.101 (PA9)
- new net UART2_RX: J2.27 (Pin_27), U4.122 (PD6)
- new net UART2_TX: J2.29 (Pin_29), U4.119 (PD5)
- new net USB_D+: R10.1, R56.1, U4.104 (PA12)
- new net USB_D-: R9.1, U4.103 (PA11)
- new net VIN: J5.1 (Pin_1)
- new net ethernet/~{CDB}: TP6.1
- new net ~{ETH_INTERRUPT}: U4.141 (PE0)
- new net ~{ETH_PME}: U4.142 (PE1)
- new net ~{ETH_RESET}: U4.118 (PD4)
- no-connect marks 0 -> 11
Other:
- removed sheet DMX
- removed sheet Digital IO
- added sheet Power Management (power.kicad_sch)
- sheet ethernet ports: added RMII_CRS_DV, RMII_REFCLKO, RMII_RX0, RMII_RX1, RMII_TX0, RMII_TX1, RMII_TXEN, SPI_CLK, SPI_MISO, SPI_MOSI, ~{CDB}, ~{INTRP}, ~{PME}, ~{RESET}, ~{SPI_CS}; removed ETH_CLK_50MHz, ETH_CRS_DV, ETH_MDC, ETH_MDIO, ETH_RXD0, ETH_RXD1, ETH_TXD0, ETH_TXD1, ETH_TX_EN
- note added: "CAN BUS"
- note added: "DEBUG"
- note added: "ETHERNET"
- note added: "FACTORY RESET SWITCH"
- note added: "I/O HEADERS"
- note added: "INDICATOR LEDS"
- note added: "MDC INTERFACE N/C IN FAVOUR OF SPI. TP LEFT IN IN CASE THIS CONFIG IS INOP"
- note added: "MICROCONTROLLER"
- note added: "NB: SPI GIVES ACCESS TO VLAN CONFIG ETC MIIM IS PHY ONLY"
- note added: "NOTE: B AKA -, A AKA +"
- note added: "NOTE: Power is not provided over USB. The device must be powered by PoE or by the VIN header in order to function"
- note added: "POWER MANAGEMENT"
- note added: "RS485"
- note added: "USB"
- moved on the sheet: H1, H2, H3, H4, J1, JP1
